File: TINY-REFLOW-CONTROLLER.sch (KiCad schematic (older format))
At the start: 51 parts, among them J1 TERMINAL-BLOCK-1x2, J2 TERMINAL-BLOCK-1x2, J3 MICRO-USB, J4 2.54mm 2x3, J5 2.54mm 1x6, M1 MOUNT_HOLE, M2 MOUNT_HOLE, M3 MOUNT_HOLE, M4 MOUNT_HOLE, M5 FIDUCIAL, M6 FIDUCIAL, Q1 2N3904, Q2 2N3904, SW1 IT-1109S, SW2 IT-1109S, SW3 TS-018, U1 ATTINY1634R-MU, U2 MCP1700T-3302E/MB, U3 MAX31856, U4 RT0802A

Commit message: Version 2.0
Parts:
- removed D2: PMEG3020CPA, RocketScreamKicadLibrary:SOT-1016, symbol DIODE_DUAL_Schottky
- removed J5: 2.54mm 1x6, RocketScreamKicadLibrary:HDR_1x6_Pitch2.54mm, symbol CONN-HDR-1x6
- removed M1, M2, M3, M4: MOUNT_HOLE, RocketScreamKicadLibrary:HOLE_NPTH_2.2MM, symbol MOUNT_HOLE
- removed M5, M6: FIDUCIAL, RocketScreamKicadLibrary:FIDUCIAL-1MM, symbol FIDUCIAL
- removed U1: ATTINY1634R-MU, RocketScreamKicadLibrary:QFN-20_4x4mm, symbol ATTINY1634_QFN
- removed U2: MCP1700T-3302E/MB, RocketScreamKicadLibrary:SOT-89, symbol MCP1700T-XXX2E/MB
- removed U4: RT0802A, RocketScreamKicadLibrary:0802A-1-SMT, symbol RT0802A
- added C13, C14, C17, C18, C19: 100nF, RocketScreamKiCadLib:C_0603, symbol RocketScreamKiCadLib:CAPACITOR-CERAMIC
- added C15, C16: 10pF, RocketScreamKiCadLib:C_0603, symbol RocketScreamKiCadLib:CAPACITOR-CERAMIC
- added F1: FUSE, RocketScreamKiCadLib:MF-FSMF, symbol RocketScreamKiCadLib:FUSE
- added J5: TERMINAL-BLOCK-1x2, RocketScreamKiCadLib:TB-1776275-2, symbol RocketScreamKiCadLib:TERMINAL-BLOCK-1x2
- added L2: LBMF1608T100K, RocketScreamKiCadLib:I_0603, symbol RocketScreamKiCadLib:INDUCTOR
- added Q3: 2N3904, RocketScreamKiCadLib:SOT-23, symbol RocketScreamKiCadLib:BJT-NPN
- added R11: 2K2, RocketScreamKiCadLib:R_0603, symbol RocketScreamKiCadLib:RESISTOR
- added R12: 53K6, RocketScreamKiCadLib:R_0603, symbol RocketScreamKiCadLib:RESISTOR
- added U1: ATMEGA328P-MU, RocketScreamKiCadLib:QFN-32_5x5mm_Pitch0.5mm, symbol RocketScreamKiCadLib:ATMEGA328P-MU
- added U2: MCP1700T-3302E-TT, RocketScreamKiCadLib:SOT-23, symbol RocketScreamKiCadLib:MCP1700T-XXX2E-TT
- added U4: CH340E, RocketScreamKiCadLib:MSOP-10, symbol RocketScreamKiCadLib:CH340E
- added U5: OLED-SSD1306-128X64-I2C, RocketScreamKiCadLib:OLED-SSD1306-128X64-I2C, symbol RocketScreamKiCadLib:OLED-SSD1306-128X64-I2C
- added Y1: NX3225GD, RocketScreamKiCadLib:NX3225GD, symbol RocketScreamKiCadLib:CRYSTAL
- C1, C2, C3, C6, C7, C8, C9: footprint RocketScreamKicadLibrary:C_0603 -> RocketScreamKiCadLib:C_0603; symbol CAPACITOR-CERAMIC -> RocketScreamKiCadLib:CAPACITOR-CERAMIC
- C10, C12: value 10uF 10V X5R -> 10uF 16V X5R; footprint RocketScreamKicadLibrary:C_0805 -> RocketScreamKiCadLib:C_0603; symbol CAPACITOR-CERAMIC -> RocketScreamKiCadLib:CAPACITOR-CERAMIC
- C11: value 10uF 10V X5R -> 100nF; footprint RocketScreamKicadLibrary:C_0805 -> RocketScreamKiCadLib:C_0603; symbol CAPACITOR-CERAMIC -> RocketScreamKiCadLib:CAPACITOR-CERAMIC
- C4: value 1uF 16V X7R -> 100nF; footprint RocketScreamKicadLibrary:C_0603 -> RocketScreamKiCadLib:C_0603; symbol CAPACITOR-CERAMIC -> RocketScreamKiCadLib:CAPACITOR-CERAMIC
- C5: value 1uF 16V X7R -> 10uF 16V X5R; footprint RocketScreamKicadLibrary:C_0603 -> RocketScreamKiCadLib:C_0603; symbol CAPACITOR-CERAMIC -> RocketScreamKiCadLib:CAPACITOR-CERAMIC
- D1: footprint RocketScreamKicadLibrary:LED_0603 -> RocketScreamKiCadLib:LED_0603; symbol LED-SINGLE -> RocketScreamKiCadLib:LED-SINGLE
- D3: footprint RocketScreamKicadLibrary:SOD-123 -> RocketScreamKiCadLib:SOD-323; symbol DIODE -> RocketScreamKiCadLib:DIODE
- J1, J2: footprint RocketScreamKicadLibrary:TB-1776275-2 -> RocketScreamKiCadLib:TB-1776275-2; symbol TERMINAL-BLOCK-1x2 -> RocketScreamKiCadLib:TERMINAL-BLOCK-1x2
- J3: footprint RocketScreamKicadLibrary:MICRO-USB -> RocketScreamKiCadLib:MICRO-USB; symbol MICRO-USB -> RocketScreamKiCadLib:MICRO-USB
- J4: footprint RocketScreamKicadLibrary:HDR_2x3_Pitch2.54mm -> RocketScreamKiCadLib:HDR_2x3_Pitch2.54mm; symbol CONN-HDR-2x3 -> RocketScreamKiCadLib:CONN-HDR-2x3
- L1: footprint RocketScreamKicadLibrary:I_0603 -> RocketScreamKiCadLib:I_0603; symbol INDUCTOR -> RocketScreamKiCadLib:INDUCTOR
- LOGO1: footprint RocketScreamKicadLibrary:LOGO-ROCKET-SCREAM_Without_Text_XXXSmall -> RocketScreamKiCadLib:LOGO-ROCKET-SCREAM_Without_Text_XXXSmall; symbol LOGO-ROCKET-SCREAM -> RocketScreamKiCadLib:LOGO-ROCKET-SCREAM-WITHOUT-TEXT
- LOGO2: footprint RocketScreamKicadLibrary:LOGO-KICAD -> RocketScreamKiCadLib:LOGO-KICAD_XSmall; symbol LOGO-KICAD -> RocketScreamKiCadLib:LOGO-KICAD
- LOGO3: footprint RocketScreamKicadLibrary:LOGO-ROCKET-SCREAM_Vertical_Medium -> RocketScreamKiCadLib:LOGO-ROCKET-SCREAM_Vertical_Small; symbol LOGO-ROCKET-SCREAM -> RocketScreamKiCadLib:LOGO-ROCKET-SCREAM-WITHOUT-TEXT
- LOGO4: footprint RocketScreamKicadLibrary:LOGO-OSHW_Small -> RocketScreamKiCadLib:LOGO-OSHW_Small; symbol LOGO-OSHW -> RocketScreamKiCadLib:LOGO-OSHW
- LS1: footprint RocketScreamKicadLibrary:HYG9605B -> RocketScreamKiCadLib:HYG9605B; symbol BUZZER -> RocketScreamKiCadLib:BUZZER
- Q1, Q2: footprint RocketScreamKicadLibrary:SOT-23 -> RocketScreamKiCadLib:SOT-23; symbol BJT-NPN -> RocketScreamKiCadLib:BJT-NPN
- R1: value 35WR10KLFTR -> 2K2; footprint RocketScreamKicadLibrary:TC33X-x -> RocketScreamKiCadLib:R_0603; symbol POTENTIOMETER -> RocketScreamKiCadLib:RESISTOR
- R10, R2, R3, R4, R5, R6, R7, R8, R9: footprint RocketScreamKicadLibrary:R_0603 -> RocketScreamKiCadLib:R_0603; symbol RESISTOR -> RocketScreamKiCadLib:RESISTOR
- SW1, SW2: footprint RocketScreamKicadLibrary:IT-1102W -> RocketScreamKiCadLib:IT-1102W; symbol TACT-SWITCH_4Pins -> RocketScreamKiCadLib:TACT-SWITCH_4Pins
- SW3: footprint RocketScreamKicadLibrary:TS-018 -> RocketScreamKiCadLib:TS-018; symbol TACT-SWITCH_2Pins -> RocketScreamKiCadLib:TACT-SWITCH_2Pins
- U3: footprint RocketScreamKicadLibrary:TSSOP-14 -> RocketScreamKiCadLib:TSSOP-14; symbol MAX31856 -> RocketScreamKiCadLib:MAX31856
Connections:
- net labels added: A0, A1, A2, A3, A6, A7, AREF, SCL, SDA
- net labels removed: D14, D15, D16, VBUS
- wire segments 166 -> 250
- no-connect marks 16 -> 8
Other:
- note added: "1. All resistor are rated 0.0625W 1% unless specified.\n2. All capacitor are rate 50 V X7R 10% unless specified."
- note added: "10mA @5.0V"
- note added: "5mA @5.0V"
- note added: "8MHz"
- note added: "ATMega328P-MU"
- note added: "Fan"
- note added: "OLED LCD"
- note added: "USB & Power Management"
- note removed: "1. All resistor are rated 0.0625W 1% unless specified.\n2. All capacitor are rate 50 V X7R 10% unless specified. \n3. "R" version of ATtiny1634 is used for better internal crystal tolerance."
- note removed: "10mA @3.3V"
- note removed: "2.2mmx4"
- note removed: "5mA @3.3V"
- note removed: "8x2 LCD"
- note removed: "ATTINY1634R"
- note removed: "FTDI Header"
- note removed: "Fiducials & Mount Holes"
- note removed: "MISO"
- note removed: "MOSI"
- note removed: "Power"
- note removed: "SCK"
- moved on the sheet: C1, C10, C11, C12, C2, C3, C4, C5, C6, C7, C8, C9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
